File: hardware/air-quality-sensor-pcb/air-quality-sensor-pcb.kicad_pcb (KiCad board)
At the start: 2 copper layers, 9 parts, among them J1 Conn_01x02, SW1 SW_Push_Dual, U1 XIAO-nRF52840-DIP, U2 Adafruit SGP40, U3 Adafruit SHT4X, U4 Adafruit BMP390, U5 Adafruit SCD4x, U6 WeAct Epaper 2.13"

Commit message: PCB decign v0.1
Parts:
- removed U6: WeAct Epaper 2.13", weact_epaper:weact_epaper_2.13
- added G***: LOGO, LOGO, F.Cu at (180.6, 68.6)
- added G***: LOGO, LOGO, F.Cu at (180.8, 61.0)
- added G***: LOGO, LOGO, F.Cu at (180.6, 72.4)
- added G***: LOGO, LOGO, F.Cu at (180.6, 64.8)
- added G***: LOGO, LOGO, F.Cu at (180.8, 76.2)
- added G***: LOGO, LOGO, F.Cu at (180.1, 55.6)
- added J2: Conn_02x04_Odd_Even, Connector_PinSocket_2.54mm:PinSocket_2x04_P2.54mm_Vertical, F.Cu at (164.1, 68.8)
- added R1: R, Resistor_THT:R_Axial_DIN0207_L6.3mm_D2.5mm_P10.16mm_Horizontal, F.Cu at (164.8, 93.0)
- added SW2: SW_DIP_x01, Button_Switch_THT:SW_DIP_SPSTx01_Slide_9.78x4.72mm_W7.62mm_P2.54mm, F.Cu at (179.3, 97.3)
- SW1: footprint Button_Switch_THT:SW_PUSH_6mm -> Button_Switch_THT:SW_PUSH-12mm
- U1: footprint Seeed_XIAO_nRF52840:XIAO-nRF52840-DIP -> seeed_xiao_nrf52:XIAO-nRF52840-DIP2
- moved U1 58.4 mm to (173.2, 117.3), turned to 180 degrees
- moved SW1 36.7 mm to (169.0, 85.2)
- moved J1 16.9 mm to (168.1, 100.1)
- moved BT1 2.12 mm to (195.8, 89.2)
- moved U5 2.12 mm to (221.2, 61.7)
- moved U2 1.99 mm to (221.2, 83.1)
- moved U4 1.83 mm to (221.2, 101.9)
- moved U3 1.69 mm to (221.2, 120.7)
Connections:
- J1 pad 2: Net-(BT1-+) -> Net-(J1-Pin_2)
- U1 pad 1: unconnected-(U1-P0.02_AIN0_LOW_A0_D0-Pad1) -> EPD_BUSY
- U1 pad 11: unconnected-(U1-P1.15_MOSI_D10-Pad11) -> SPI_SDA
- U1 pad 2: unconnected-(U1-P0.03_AIN1_LOW_A1_D1-Pad2) -> EPD_RES
- U1 pad 3: unconnected-(U1-P0.28_AIN4_LOW_A2_D2-Pad3)_1 -> EPD D/C
- U1 pad 4: unconnected-(U1-P0.29_AIN5_LOW_A3_D3-Pad4)_1 -> EPD CS
- U1 pad 5: unconnected-(U1-P0.04_AIN2_A4_D4-Pad5) -> I2C_SDA
- U1 pad 6: unconnected-(U1-P0.05_AIN3_A5_D5-Pad6) -> I2C_SCL
- U1 pad 8: unconnected-(U1-P1.12_RX_D7-Pad8) -> Button
- U1 pad 9: unconnected-(U1-P1.13_SCK_D8-Pad9)_1 -> SPI_SCL
- U2 pad 4: SCL -> I2C_SCL
- U2 pad 5: SDA -> I2C_SDA
- U3 pad 4: SCL -> I2C_SCL
- U3 pad 5: SDA -> I2C_SDA
- U4 pad 4: SCL -> I2C_SCL
- U4 pad 6: SDA -> I2C_SDA
- U5 pad 4: SCL -> I2C_SCL
- U5 pad 5: SDA -> I2C_SDA
Routing:
- net I2C_SDA: track 0.00 -> 104.4 mm, vias 0 -> 1
- net I2C_SCL: track 0.00 -> 100.3 mm, vias 0 -> 1
- net Net-(BT1--): track 0.00 -> 66.7 mm, vias 0 -> 2
- net EPD_BUSY: track 0.00 -> 63.1 mm
- net SPI_SDA: track 0.00 -> 62.4 mm, vias 0 -> 1
- net EPD D/C: track 0.00 -> 62.3 mm, vias 0 -> 1
- net EPD_RES: track 0.00 -> 60.0 mm
- net EPD CS: track 0.00 -> 57.5 mm
- net SPI_SCL: track 0.00 -> 55.5 mm
- net Button: track 0.00 -> 43.6 mm
- net Net-(BT1-+): track 0.00 -> 27.8 mm, vias 0 -> 1
- net Net-(J1-Pin_2): track 0.00 -> 19.6 mm
- added copper zone on F.Cu, net +3V3
- added copper zone on B.Cu, net GND
Other:
- board outline added: 72.9 x 80.3 mm
- board text added: "3V3"
- board text added: "Air quality monitor Version 0.1 Paavo Palomäki 05/2025"
- board text added: "BUSY"
- board text added: "CS"
- board text added: "D/C"
- board text added: "E-paper display connector"
- board text added: "GND"
- board text added: "RES"
- board text added: "SCL"
- board text added: "SDA"
